File: Eagle/NANDgate.brd (EAGLE design)
At the start: 72 x 48 mm, 12 parts, among them IC1 74LVC1G00DBV

Commit message: updated for v1.3
Routing:
- net Y: track 55.1 -> 57.7 mm
Other:
- board text added: "JLCJLCJLCJLC"
- board text added: "LogicBits v1.3 by Alexander Kirillov github.com/shurik179"
- board text removed: "LogicBits v1.2 by Alexander Kirillov github.com/shurik179"
Changed lines of the file:
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@@
 <circle x="52" y="0" radius="2" width="1" layer="22"/>
 <circle x="36" y="13" radius="9" width="0.1" layer="21"/>
-<text x="52" y="-20" size="1.778" layer="21" rot="SR90">LogicBits v1.2 by Alexander Kirillov
+<text x="52" y="-20" size="1.778" layer="21" rot="SR90">LogicBits v1.3 by Alexander Kirillov
 github.com/shurik179</text>
 <wire x1="2" y1="12" x2="0" y2="12" width="1" layer="22"/>
@@
 <wire x1="72" y1="4" x2="69" y2="4" width="0.2" layer="22"/>
 <wire x1="72" y1="-4" x2="69" y2="-4" width="0.2" layer="22"/>
+<text x="28" y="12" size="1.778" layer="21">JLCJLCJLCJLC</text>
 </plain>
 <attributes>
@@
 <wire x1="56" y1="1.25" x2="54.75" y2="2.5" width="0.25" layer="1"/>
 <wire x1="54.75" y1="2.5" x2="54.75" y2="7.75" width="0.25" layer="1"/>
-<wire x1="54.75" y1="7.75" x2="55.46" y2="8.46" width="0.25" layer="1"/>
+<wire x1="55.46" y1="8.46" x2="54.75" y2="7.75" width="0.25" layer="1"/>
 <contactref element="IC1" pad="4"/>
 <wire x1="26.3" y1="-1.95" x2="28.3501" y2="-1.95" width="0.25" layer="1"/>
 <wire x1="28.3501" y1="-1.95" x2="28.3601" y2="-1.94" width="0.25" layer="1"/>
 <contactref element="JP4" pad="1"/>
-<wire x1="55.46" y1="8.46" x2="58" y2="8.46" width="0" layer="19" extent="1-1"/>
+<wire x1="58" y1="8.46" x2="55.46" y2="8.46" width="0.25" layer="1"/>
 </signal>
 <signal name="N$1">
