File: Eagle/NOTgate.brd (EAGLE design)
At the start: 72 x 48 mm, 9 parts, among them IC1 74LVC1G14DBV

Commit message: updated for v1.3
Routing:
- net VCC: track 64.3 -> 65.5 mm
Other:
- board text added: "JLCJLCJLCJLC"
- board text added: "LogicBits v1.3 by Alexander Kirillov github.com/shurik179"
- board text removed: "LogicBits v1.2 by Alexander Kirillov github.com/shurik179"
Changed lines of the file:
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@@
 <text x="29" y="0" size="8" layer="22" ratio="12" rot="SMR180" align="center">NOT</text>
 <circle x="36" y="13" radius="9" width="0.1" layer="21"/>
-<text x="52" y="-20" size="1.778" layer="21" rot="SR90">LogicBits v1.2 by Alexander Kirillov
+<text x="52" y="-20" size="1.778" layer="21" rot="SR90">LogicBits v1.3 by Alexander Kirillov
 github.com/shurik179</text>
 <wire x1="0" y1="0" x2="2" y2="0" width="1" layer="22"/>
@@
 <wire x1="70" y1="4" x2="72" y2="4" width="0.2" layer="22"/>
 <wire x1="70" y1="-4" x2="72" y2="-4" width="0.2" layer="22"/>
+<text x="28" y="12" size="1.778" layer="21">JLCJLCJLCJLC</text>
 </plain>
 <attributes>
@@
 <contactref element="JP3" pad="2"/>
 <contactref element="JP2" pad="2"/>
-<wire x1="26.4001" y1="0" x2="53" y2="0" width="0.5" layer="1"/>
 <wire x1="53" y1="0" x2="58" y2="0" width="0.5" layer="1"/>
 <contactref element="JP4" pad="2"/>
@@
 <wire x1="53" y1="9" x2="53" y2="0" width="0.5" layer="1"/>
 <wire x1="19" y1="0" x2="20" y2="1" width="0.5" layer="1"/>
-<wire x1="20" y1="1" x2="25" y2="1" width="0.5" layer="1"/>
-<wire x1="25" y1="1" x2="26" y2="0" width="0.5" layer="1"/>
-<wire x1="26" y1="0" x2="26" y2="-0.04" width="0.5" layer="1"/>
 <wire x1="14" y1="0" x2="19" y2="0" width="0.5" layer="1"/>
-<wire x1="25.96" y1="-0.04" x2="25" y2="-1" width="0.25" layer="1"/>
-<wire x1="25" y1="-1" x2="25" y2="-3" width="0.25" layer="1"/>
+<wire x1="25" y1="-3" x2="25" y2="-1" width="0.25" layer="1"/>
 <wire x1="25" y1="-3" x2="24" y2="-4" width="0.25" layer="1"/>
 <wire x1="24" y1="-4" x2="23.762" y2="-4" width="0.25" layer="1"/>
 <contactref element="IC1" pad="5"/>
-<wire x1="26.3" y1="-0.05" x2="26.4001" y2="0" width="0" layer="19" extent="1-1"/>
-<wire x1="26" y1="-0.04" x2="26.3" y2="-0.05" width="0" layer="19" extent="1-1"/>
-<wire x1="25.96" y1="-0.04" x2="26" y2="-0.04" width="0" layer="19" extent="1-1"/>
+<wire x1="26.3" y1="-0.05" x2="26.35" y2="0" width="0.5" layer="1"/>
+<wire x1="26.35" y1="0" x2="53" y2="0" width="0.5" layer="1"/>
+<wire x1="26" y1="1" x2="26.35" y2="0.65" width="0.5" layer="1"/>
+<wire x1="26.35" y1="0.65" x2="26.35" y2="0" width="0.5" layer="1"/>
+<wire x1="20" y1="1" x2="26" y2="1" width="0.5" layer="1"/>
+<wire x1="25" y1="-1" x2="25.95" y2="-0.05" width="0.25" layer="1"/>
+<wire x1="25.95" y1="-0.05" x2="26.3" y2="-0.05" width="0.25" layer="1"/>
 </signal>
 <signal name="N$3">
