File: Eagle/ORgate.brd (EAGLE design)
At the start: 72 x 48 mm, 12 parts, among them IC1 74AHC1G32DBV

Commit message: updated for v1.3
Other:
- board text added: "JLCJLCJLCJLC"
- board text added: "LogicBits v1.3 by Alexander Kirillov github.com/shurik179"
- board text removed: "LogicBits v1.2 by Alexander Kirillov github.com/shurik179"
