File: Eagle/XORgate.brd (EAGLE design)
At the start: 72 x 48 mm, 12 parts, among them IC1 74AHC1G86DBV

Commit message: updated for v1.3
Other:
- board text added: "JLCJLCJLCJLC"
Changed lines of the file:
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@@
 <wire x1="72" y1="4" x2="70" y2="4" width="0.2" layer="22"/>
 <wire x1="72" y1="-4" x2="70" y2="-4" width="0.2" layer="22"/>
+<text x="28" y="12" size="1.778" layer="21">JLCJLCJLCJLC</text>
 </plain>
 <attributes>
